Commit message: ROS2 cam

File: ROS2/lab-ws/src/labbot_description/urdf/description.urdf.xacro (robot description, xacro)
@@ -129,4 +129,5 @@
     </link>
     <link name="rgb_camera">
+        <xacro:default_inertial mass="0.001"/>
         <visual>
             <origin rpy="-1.57 0 -1.57" xyz="-0.1 0.125 0.15"/>
@@ -135,4 +136,10 @@
             </geometry>
         </visual>
+        <collision>
+            <origin rpy="-1.57 0 -1.57" xyz="-0.1 0.125 0.15"/>
+            <geometry>
+                <mesh filename="package://arduinobot_description/meshes/pi_camera.STL" scale="0.01 0.01 0.01"/>
+            </geometry>
+        </collision>
     </link>
     <!-- Joints -->
@@ -193,3 +200,28 @@
         <origin xyz="0 0.45 0.2" rpy="0 -0.5 1.57"/>
     </joint>
+    <gazebo reference="rgb_camera">
+        <sensor name="camera" type="camera">
+            <always_on>true</always_on>
+            <update_rate>30.0</update_rate>
+            <visualize>true</visualize>
+            <topic>image_raw</topic>
+            <gz_frame_id>rgb_camera</gz_frame_id>
+            <camera name="camera">
+            <horizontal_fov>1.21126</horizontal_fov>
+            <image>
+                <width>2304</width>
+                <height>1296</height>
+                <format>R8G8B8</format>
+            </image>
+            <distortion>
+                <k1>0.0</k1>
+                <k2>0.0</k2>
+                <k3>0.0</k3>
+                <p1>0.0</p1>
+                <p2>0.0</p2>
+                <center>0.5 0.5</center>
+            </distortion>
+            </camera>
+        </sensor>
+    </gazebo>
 </robot>

File: ROS2/lab-ws/src/labbot_description/urdf/gazebo.xacro (robot description, xacro)
@@ -1,5 +1,4 @@
 <?xml version="1.0"?>
 <robot xmlns:xacro="http://www.ros.org/wiki/xacro" name="arduinobot">
-  <!-- ROS 2 Control -->
   <gazebo>
     <!-- ROS 2 Humble -->
@@ -7,4 +6,7 @@
       <plugin filename="ign_ros2_control-system" name="ign_ros2_control::IgnitionROS2ControlPlugin">
         <!-- <parameters>$(find arduinobot_controller)/config/arduinobot_controllers.yaml</parameters> -->
+      </plugin>
+      <plugin filename="ignition-gazebo-sensors-system" name="ignition::gazebo::systems::Sensors">
+        <render_engine>ogre2</render_engine>
       </plugin>
     </xacro:if>
@@ -14,4 +16,7 @@
         <!-- <parameters>$(find arduinobot_controller)/config/arduinobot_controllers.yaml</parameters> -->
       </plugin>
+      <plugin filename="gz-sim-sensors-system" name="gz::sim::systems::Sensors">
+        <render_engine>ogre2</render_engine>
+      </plugin>
     </xacro:unless>
   </gazebo>
